Commit message: working version without collision

File: models/franka_description/robots/panda_arm_hand_cam_closed.urdf (robot description, URDF)
Before this commit: robot panda, 14 links, 13 joints
Joints:
- joint panda_finger_joint1: origin xyz=0.00000 -0.05000 0.05840 rpy=0.00000 -0.00000 0.00000 -> xyz=0.00000 -0.00000 0.05840 rpy=0.00000 -0.00000 0.00000
- joint panda_finger_joint2: origin xyz=0.00000 0.05000 0.05840 rpy=0.00000 -0.00000 0.00000 -> xyz=0.00000 0.00000 0.05840 rpy=0.00000 -0.00000 0.00000
